File: pcb/ayrton-mainboard/psu.kicad_sch (KiCad schematic)
At the start: 78 parts, among them J2 CONN_PCIE_PWR_8PIN, J3 CONN_IBC_MGMT, U10 MYMGK00506ERSR, U4 LP2996A, U5 MYMGK1R812ERSR, U6 MYMGK00506ERSR, U7 MYMGK00504ERSR, U8 MYMGK00504ERSR, U9 MYMGK00504ERSR

Commit message: Continued initial schematic, working on LPDDR4
Parts:
- removed C41: 47 uF, azonenberg_pcb:EIA_0805_CAP_NOSILK, symbol device:C
- removed C42, C46: 0.1 uF, azonenberg_pcb:EIA_0402_CAP_NOSILK, symbol device:C
- removed C43, C49: 0.47 uF, azonenberg_pcb:EIA_0402_CAP_NOSILK, symbol device:C
- removed C44: 47 uF, azonenberg_pcb:EIA_1206_CAP_NOSILK, symbol device:C
- removed C45, C48, C59, C60, C61, C62, C78, C79, C80, C81: 100 uF, azonenberg_pcb:EIA_1210_CAP_NOSILK, symbol device:C
- removed C47: 4.7 uF, azonenberg_pcb:EIA_0603_CAP_NOSILK, symbol device:C
- removed C50, C51, C57, C58, C63, C64, C67, C68, C72, C73, C74, C75: 22 uF 25V, azonenberg_pcb:EIA_1812_CAP_NOSILK, symbol device:C
- removed C52, C53, C54, C65, C66, C69, C70, C76, C77: 220 uF, azonenberg_pcb:EIA_1210_CAP_NOSILK, symbol device:C
- removed C55: 0.47 uF, symbol device:C
- removed C71: DNP, azonenberg_pcb:EIA_1210_CAP_NOSILK, symbol device:C
- removed R10: 4.7k, azonenberg_pcb:EIA_0402_RES_NOSILK, symbol device:R
- removed R11: 300, azonenberg_pcb:EIA_0402_RES_NOSILK, symbol device:R
- removed R12, R17, R18, R6: 0, azonenberg_pcb:EIA_0402_RES_NOSILK, symbol passive-azonenberg:R_PWR
- removed R13: 2.2k, azonenberg_pcb:EIA_0402_RES_NOSILK, symbol device:R
- removed R14: 22, azonenberg_pcb:EIA_0402_RES_NOSILK, symbol device:R
- removed R15: 10K, azonenberg_pcb:EIA_0402_RES_NOSILK, symbol device:R
- removed R16, R19, R3, R5, R7: 0, azonenberg_pcb:EIA_0402_RES_NOSILK, symbol device:R
- removed R2: 100, azonenberg_pcb:EIA_0402_RES_NOSILK, symbol device:R
- removed R20, R21, R8, R9: FIXME, azonenberg_pcb:EIA_0402_RES_NOSILK, symbol device:R
- removed R4: 16K, azonenberg_pcb:EIA_0402_RES_NOSILK, symbol device:R
- removed TP1, TP2, TP3, TP4, TP5, TP6: TESTPOINT, azonenberg_pcb:TESTPOINT_SMT_0.5MM, symbol conn:CONN_01X01
- removed U10, U6: MYMGK00506ERSR, azonenberg_pcb:MODULE_MURATA_MYMGK00504ERSR, symbol power-azonenberg:MYMGK00504ERSR
- removed U4: LP2996A, azonenberg_pcb:SOIC_8_3.9MM_EPAD, symbol power-azonenberg:LP2996A
- removed U5: MYMGK1R812ERSR, azonenberg_pcb:MODULE_MURATA_MYMGK1R812, symbol power-azonenberg:MYMGK1R812ERSR
- removed U7, U8, U9: MYMGK00504ERSR, azonenberg_pcb:MODULE_MURATA_MYMGK00504ERSR, symbol power-azonenberg:MYMGK00504ERSR
Other:
- added sheet 0.x V rails (0vx.kicad_sch)
- added sheet 1.x V rails (1vx.kicad_sch)
- added sheet 2V and higher rails (higher-voltage.kicad_sch)
- added sheet Supervisor (super.kicad_sch)
- note added: "IBC power and data connections"
- note removed: "1.8V Vih Internal: 33K pulldown, 100K pullup So should float at ~2.7V if undriven"
- note removed: "PGOOD pin for all MYMGK1R812 rails (VCCINT, GTY_VTT) is pulled up to 5V internally, need to be on 5V tolerant pin. Other regs have external pullups to 3V3_SB"
- note removed: "Total output C 400 - 3000 uF"
- note removed: "Total output C 660 - 5000 uF"
- note removed: "Trim: Precision metal film 1/10W +/- 0.5%"
