File: pcb/ayrton-mainboard/soc-ram.kicad_sch (KiCad schematic)
At the start: 1 part, among them U1 STM32MP257FAI3

Commit message: Continued initial system design
Other:
- moved on the sheet: U1F
Changed lines of the file:
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@@
 	(title_block
 		(title "AYRTON Main Board")
-		(date "2024-11-15")
+		(date "2024-11-18")
 		(rev "0.1")
 		(company "Antikernel Labs")
 		(comment 1 "Andrew D. Zonenberg")
 	)
+	(hierarchical_label "GND"
+		(shape input)
+		(at 72.39 135.89 0)
+		(fields_autoplaced yes)
+		(effects
+			(font
+				(size 1.27 1.27)
+			)
+			(justify left)
+		)
+	)
+	(hierarchical_label "1V1"
+		(shape input)
+		(at 73.66 129.54 0)
+		(fields_autoplaced yes)
+		(effects
+			(font
+				(size 1.27 1.27)
+			)
+			(justify left)
+		)
+	)
+	(hierarchical_label "1V8"
+		(shape input)
+		(at 83.82 124.46 0)
+		(fields_autoplaced yes)
+		(effects
+			(font
+				(size 1.27 1.27)
+			)
+			(justify left)
+		)
+	)
 	(symbol
 		(lib_id "st-azonenberg:STM32MP257FAI3")
-		(at 138.43 130.81 0)
+		(at 143.51 110.49 0)
 		(unit 6)
 		(exclude_from_sim no)
@@
 		(on_board yes)
 		(dnp no)
-		(fields_autoplaced yes)
 		(property "Reference" "U1"
-			(at 153.035 45.5125 0)
+			(at 143.51 111.8757 0)
 			(effects
 				(font
 					(size 1.27 1.27)
 				)
+				(justify left)
 			)
 		)
 		(property "Value" "STM32MP257FAI3"
-			(at 153.035 47.9368 0)
+			(at 143.51 114.3 0)
 			(effects
 				(font
 					(size 1.27 1.27)
 				)
+				(justify left)
 			)
 		)
 		(property "Footprint" ""
-			(at 138.43 130.81 0)
+			(at 143.51 110.49 0)
 			(effects
 				(font
@@
 		)
 		(property "Datasheet" ""
-			(at 138.43 130.81 0)
+			(at 143.51 110.49 0)
 			(effects
 				(font
@@
 		)
 		(property "Description" ""
-			(at 138.43 130.81 0)
+			(at 143.51 110.49 0)
 			(effects
 				(font
@@
 		)
 		(pin "K3"
+			(alternate "TRACECLK")
 		)
 		(pin "W10"
@@
 		)
 		(pin "H1"
+			(alternate "TRACED1")
 		)
 		(pin "M3"
@@
 		)
 		(pin "L1"
+			(alternate "TRACED3")
 		)
 		(pin "E17"
@@
 		)
 		(pin "L4"
+			(alternate "TRACED0")
 		)
 		(pin "U19"
@@
 		)
 		(pin "L7"
+			(alternate "TRACED2")
 		)
 		(pin "V11"
@@
 		(on_board yes)
 		(dnp no)
-		(fields_autoplaced yes)
 		(property "Reference" "U1"
-			(at 86.995 67.3678 0)
+			(at 71.12 109.3357 0)
 			(effects
 				(font
@@
 		)
 		(property "Value" "STM32MP257FAI3"
-			(at 86.995 69.7921 0)
+			(at 71.12 111.76 0)
 			(effects
 				(font
@@
 		)
 		(pin "K3"
+			(alternate "TRACECLK")
 		)
 		(pin "W10"
@@
 		)
 		(pin "H1"
+			(alternate "TRACED1")
 		)
 		(pin "M3"
@@
 		)
 		(pin "L1"
+			(alternate "TRACED3")
 		)
 		(pin "E17"
@@
 		)
 		(pin "L4"
+			(alternate "TRACED0")
 		)
 		(pin "U19"
@@
 		)
 		(pin "L7"
+			(alternate "TRACED2")
 		)
 		(pin "V11"

Commit message: Continued initial schematic, working on LPDDR4
Parts:
- added C176, C177, C198, C203, C208, C209: 4.7 uF, symbol device:C
- added C178, C179, C180, C181, C182, C183, C184, C185, C186, C187, C188, C189, C190, C191, C192, C193, C194, C195, C196, C197, C199, C200, C201, C202, C204, C205, C206, C207, C210, C211, C212, C213, C214, C215, C216, C217, C218, C219, C220, C221, C222, C223, C224, C225, C226, C227, C228, C229, C230, C231, C232, C233: 0.47 uF, symbol device:C
- added R81, R83: 240, symbol device:R
- added R82: 10K, symbol device:R
- added R84: DNP, symbol device:R
- added U18: B1621PM2FDGUK-U, symbol memory-azonenberg:LPDDR4_X16_DUALCHANNEL
Connections:
- net 1V1: now also C176.1, C177.1, C178.1, C179.1, C180.1, C181.1, C182.1, C183.1, C184.1, C185.1, C186.1, C187.1, C188.1, C189.1, C190.1, C191.1, C192.1, C193.1, C194.1, C195.1, C196.1, C197.1, C208.1, C209.1, C210.1, C211.1, C212.1, C213.1, C214.1, C215.1, C216.1, C217.1, C218.1, C219.1, C220.1, C221.1, C222.1, C223.1, C224.1, C225.1, C226.1, C227.1, C228.1, C229.1, C230.1, C231.1, C232.1, C233.1, R83.1, R84.1, U18.A4 (VDD2), U18.A9 (VDD2), U18.AA10 (VDDQ), U18.AA3 (VDDQ), U18.AA5 (VDDQ), U18.AA8 (VDDQ), U18.AB4 (VDD2), U18.AB9 (VDD2), U18.B19 (VDDQ), U18.B3 (VDDQ), U18.B5 (VDDQ), U18.B8 (VDDQ), U18.D1 (VDDQ), U18.D12 (VDDQ), U18.D5 (VDDQ), U18.D8 (VDDQ), U18.F10 (VDDQ), U18.F3 (VDDQ), U18.F5 (VDD2), U18.F8 (VDD2), U18.G2 (ODT_CA_A), U18.H1 (VDD2), U18.H12 (VDD2), U18.H5 (VDD2), U18.H8 (VDD2), U18.K1 (VDD2), U18.K10 (VDD2), U18.K12 (VDD2), U18.K3 (VDD2), U18.N1 (VDD2), U18.N10 (VDD2), U18.N12 (VDD2), U18.N3 (VDD2), U18.R1 (VDD2), U18.R12 (VDD2), U18.R5 (VDD2), U18.R8 (VDD2), U18.T2 (ODT_CA_B), U18.U10 (VDDQ), U18.U3 (VDDQ), U18.U5 (VDD2), U18.U8 (VDD2), U18.W1 (VDDQ), U18.W12 (VDDQ), U18.W5 (VDDQ), U18.W8 (VDDQ)
- net 1V8: now also C198.1, C199.1, C200.1, C201.1, C202.1, C203.1, C204.1, C205.1, C206.1, C207.1, U18.F1 (VDD1), U18.F12 (VDD1), U18.G4 (VDD1), U18.G9 (VDD1), U18.T4 (VDD1), U18.T9 (VDD1), U18.U1 (VDD1), U18.U12 (VDD1)
- net GND: now also C176.2, C177.2, C178.2, C179.2, C180.2, C181.2, C182.2, C183.2, C184.2, C185.2, C186.2, C187.2, C188.2, C189.2, C190.2, C191.2, C192.2, C193.2, C194.2, C195.2, C196.2, C197.2, C198.2, C199.2, C200.2, C201.2, C202.2, C203.2, C204.2, C205.2, C206.2, C207.2, C208.2, C209.2, C210.2, C211.2, C212.2, C213.2, C214.2, C215.2, C216.2, C217.2, C218.2, C219.2, C220.2, C221.2, C222.2, C223.2, C224.2, C225.2, C226.2, C227.2, C228.2, C229.2, C230.2, C231.2, C232.2, C233.2, R81.2, R82.2, U18.A10 (VSS), U18.A3 (VSS), U18.AB10 (VSS), U18.AB3 (VSS), U18.AB5 (VSS), U18.AB8 (VSS), U18.C1 (VSS), U18.C12 (VSS), U18.C5 (VSS), U18.C8 (VSS), U18.D11 (VSS), U18.D2 (VSS), U18.D4 (VSS), U18.D9 (VSS), U18.E1 (VSS), U18.E12 (VSS), U18.E5 (VSS), U18.E8 (VSS), U18.G1 (VSS), U18.G10 (VSS), U18.G12 (VSS), U18.G3 (VSS), U18.G5 (VSS), U18.G8 (VSS), U18.J1 (VSS), U18.J10 (VSS), U18.J12 (VSS), U18.J3 (VSS), U18.K11 (VSS), U18.K2 (VSS), U18.K4 (VSS), U18.K9 (VSS), U18.N11 (VSS), U18.N2 (VSS), U18.N4 (VSS), U18.N9 (VSS), U18.P1 (VSS), U18.P10 (VSS), U18.P12 (VSS), U18.P3 (VSS), U18.T1 (VSS), U18.T10 (VSS), U18.T12 (VSS), U18.T3 (VSS), U18.T5 (VSS), U18.T8 (VSS), U18.V1 (VSS), U18.V12 (VSS), U18.V5 (VSS), U18.V8 (VSS), U18.W11 (VSS), U18.W2 (VSS), U18.W4 (VSS), U18.W9 (VSS), U18.Y1 (VSS), U18.Y12 (VSS), U18.Y5 (VSS), U18.Y8 (VSS)
- net LPDDR4_CHA_DQ3: now reaches U1.AA22 (DDR_DQ3)
- net LPDDR4_CHA_DQ3: now also U18.F2 (DQ3_A)
- net LPDDR4_CHB_DQ3: now reaches U1.B22 (DDR_DQ19)
- net LPDDR4_CHB_DQ3: now also U18.U2 (DQ3_B)
- net LPDDR4_CHB_DQ2: now reaches U1.C21 (DDR_DQ18)
- net LPDDR4_CHB_DQ2: now also U18.V2 (DQ2_B)
- net LPDDR4_CHB_DQ1: now reaches U1.C22 (DDR_DQ17)
- net LPDDR4_CHB_DQ1: now also U18.Y2 (DQ1_B)
- net LPDDR4_CHB_DQ0: now reaches U1.D20 (DDR_DQ16)
- net LPDDR4_CHB_DQ0: now also U18.AA2 (DQ0_B)
- net LPDDR4_DHB_DQS0_P: now reaches U1.D21 (DDR_DQS2_P)
- net LPDDR4_DHB_DQS0_P: now also U18.W3 (DQS0_B_P)
- net LPDDR4_DHB_DQS0_N: now reaches U1.D22 (DDR_DQS2_N)
- net LPDDR4_DHB_DQS0_N: now also U18.V3 (DQS0_B_N)
- net LPDDR4_CHB_DQ6: now reaches U1.E19 (DDR_DQ22)
- net LPDDR4_CHB_DQ6: now also U18.Y4 (DQ6_B)
- net LPDDR4_CHB_DQ7: now reaches U1.E20 (DDR_DQ23)
- net LPDDR4_CHB_DQ7: now also U18.AA4 (DQ7_B)
- net LPDDR4_CHB_DMI0: now reaches U1.E21 (DDR_DQM2)
- net LPDDR4_CHB_DMI0: now also U18.Y3 (DMI0_B)
- net LPDDR4_RST_N: now reaches U1.F18 (DDR_RESETN)
- net LPDDR4_RST_N: now also R82.1, U18.T11 (RESET_N)
- net LPDDR4_CHB_DQ5: now reaches U1.F19 (DDR_DQ21)
- net LPDDR4_CHB_DQ5: now also U18.V4 (DQ5_B)
- net LPDDR4_CHB_DQ4: now reaches U1.F20 (DDR_DQ20)
- net LPDDR4_CHB_DQ4: now also U18.U4 (DQ4_B)
- net LPDDR4_CHB_DQ8: now reaches U1.G19 (DDR_DQ24)
- net LPDDR4_CHB_DQ8: now also U18.AA11 (DQ8_B)
- net LPDDR4_CHB_DQ11: now reaches U1.G20 (DDR_DQ27)
- net LPDDR4_CHB_DQ11: now also U18.U11 (DQ11_B)
- net LPDDR4_CHB_DQ10: now reaches U1.G21 (DDR_DQ26)
- net LPDDR4_CHB_DQ10: now also U18.V11 (DQ10_B)
- net LPDDR4_CHB_DQ9: now reaches U1.G22 (DDR_DQ25)
- net LPDDR4_CHB_DQ9: now also U18.Y11 (DQ9_B)
- net LPDDR4_CHB_DMI1: now reaches U1.H20 (DDR_DQM3)
- net LPDDR4_CHB_DMI1: now also U18.Y10 (DMI1_B)
- net LPDDR4_CHB_DQS1_N: now reaches U1.H21 (DDR_DQS3_N)
- net LPDDR4_CHB_DQS1_N: now also U18.V10 (DQS1_B_N)
- net LPDDR4_CHB_DQS1_P: now reaches U1.H22 (DDR_DQS3_P)
- net LPDDR4_CHB_DQS1_P: now also U18.W10 (DQS1_B_P)
- net LPDDR4_CHB_DQ13: now reaches U1.J20 (DDR_DQ29)
- net LPDDR4_CHB_DQ13: now also U18.V9 (DQ13_B)
- net LPDDR4_CHB_DQ12: now reaches U1.J21 (DDQ_DQ28)
- net LPDDR4_CHB_DQ12: now also U18.U9 (DQ12_B)
- net LPDDR4_SOC_RZQ: now reaches U1.K16 (DDR_ZQ)
- net LPDDR4_SOC_RZQ: now also R81.1
- net LPDDR4_CHB_DQ14: now reaches U1.K20 (DDR_DQ30)
- net LPDDR4_CHB_DQ14: now also U18.Y9 (DQ14_B)
- net LPDDR4_CHB_DQ15: now reaches U1.L19 (DDR_DQ31)
- net LPDDR4_CHB_DQ15: now also U18.AA9 (DQ15_B)
- net LPDDR4_CHA_DQ10: now reaches U1.L21 (DDR_DQ10)
- net LPDDR4_CHA_DQ10: now also U18.E11 (DQ10_A)
- net LPDDR4_CHA_DQ11: now reaches U1.L22 (DDR_DQ11)
- net LPDDR4_CHA_DQ11: now also U18.F11 (DQ11_A)
- net LPDDR4_CHA_DQ8: now reaches U1.M21 (DDR_DQ8)
- net LPDDR4_CHA_DQ8: now also U18.B11 (DQ8_A)
- net LPDDR4_CHA_DQ9: now reaches U1.M22 (DDR_DQ9)
- net LPDDR4_CHA_DQ9: now also U18.C11 (DQ9_A)
- net LPDDR4_CHA_DQS1_P: now reaches U1.N20 (DDR_DQS1_P)
- net LPDDR4_CHA_DQS1_P: now also U18.D10 (DQS1_A_P)
- net LPDDR4_CHA_DQS1_N: now reaches U1.N21 (DDR_DQS1_N)
- net LPDDR4_CHA_DQS1_N: now also U18.E10 (DQS1_A_N)
- net LPDDR4_CHA_DMI1: now reaches U1.P20 (DDR_DQM1)
- net LPDDR4_CHA_DMI1: now also U18.C10 (DMI1_A)
- net LPDDR4_CHA_DQ13: now reaches U1.R20 (DDR_DQ13)
- net LPDDR4_CHA_DQ13: now also U18.E9 (DQ13_A)
- net LPDDR4_CHA_DQ14: now reaches U1.R21 (DDR_DQ14)
- net LPDDR4_CHA_DQ14: now also U18.C9 (DQ14_A)
- net LPDDR4_CHA_DQ15: now reaches U1.R22 (DDR_DQ15)
- net LPDDR4_CHA_DQ15: now also U18.B9 (DQ15_A)
- net LPDDR4_CHA_DQ5: now reaches U1.T20 (DDR_DQ5)
- net LPDDR4_CHA_DQ5: now also U18.E4 (DQ5_A)
- net LPDDR4_CHA_DQ4: now reaches U1.T21 (DDR_DQ4)
- net LPDDR4_CHA_DQ4: now also U18.F4 (DQ4_A)
- net LPDDR4_CHA_DQ12: now reaches U1.T22 (DDR_DQ12)
- net LPDDR4_CHA_DQ12: now also U18.F9 (DQ12_A)
- net LPDDR4_CHA_DQ7: now reaches U1.U20 (DDR_DQ7)
- net LPDDR4_CHA_DQ7: now also U18.B4 (DQ7_A)
- net LPDDR4_CHA_DQ6: now reaches U1.U21 (DDR_DQ6)
- net LPDDR4_CHA_DQ6: now also U18.C4 (DQ6_A)
- net LPDDR4_CHA_DQS0_P: now reaches U1.V20 (DDR_DQS0_P)
- net LPDDR4_CHA_DQS0_P: now also U18.D3 (DQS0_A_P)
- net LPDDR4_CHA_DQS0_N: now reaches U1.W20 (DDR_DQS0_N)
- net LPDDR4_CHA_DQS0_N: now also U18.E3 (DQS0_A_N)
- net LPDDR4_CHA_DMI0: now reaches U1.W21 (DDR_DQM0)
- net LPDDR4_CHA_DMI0: now also U18.C3 (DMI0_A)
- net LPDDR4_CHA_DQ0: now reaches U1.W22 (DDR_DQ0)
- net LPDDR4_CHA_DQ0: now also U18.B2 (DQ0_A)
- net LPDDR4_CHA_DQ1: now reaches U1.Y21 (DDR_DQ1)
- net LPDDR4_CHA_DQ1: now also U18.C2 (DQ1_A)
- net LPDDR4_CHA_DQ2: now reaches U1.Y22 (DDR_DQ2)
- net LPDDR4_CHA_DQ2: now also U18.E2 (DQ2_A)
- net LPDDR4_CHB_CA_2: now reaches U1.G18 (DDR_A20)
- net LPDDR4_CHB_CA_2: now also U18.R9 (CA2_B)
- net LPDDR4_CHB_CA_4: now reaches U1.H17 (DDR_A22)
- net LPDDR4_CHB_CA_4: now also U18.R11 (CA4_B)
- net LPDDR4_CHB_CLK_N: now reaches U1.H18 (DDR_A17)
- net LPDDR4_CHB_CLK_N: now also U18.P9 (CLK_B_N)
- net LPDDR4_CHB_CS_N: now reaches U1.H19 (DDR_A18)
- net LPDDR4_CHB_CS_N: now also U18.R4 (CS0_B)
- net LPDDR4_CHB_CA_5: now reaches U1.J17 (DDR_A23)
- net LPDDR4_CHB_CA_5: now also U18.P11 (CA5_B)
- net LPDDR4_CHB_CLK_P: now reaches U1.J18 (DDR_A16)
- net LPDDR4_CHB_CLK_P: now also U18.P8 (CLK_B_P)
- net LPDDR4_CHB_CA_3: now reaches U1.J19 (DDR_A21)
- net LPDDR4_CHB_CA_3: now also U18.R10 (CA3_B)
- net LPDDR4_CHB_CKE: now reaches U1.K19 (DDR_A12)
- net LPDDR4_CHB_CKE: now also U18.P4 (CKE0_B)
- net LPDDR4_CHB_CA_1: now reaches U1.L17 (DDR_A15)
- net LPDDR4_CHB_CA_1: now also U18.P2 (CA1_B)
- net LPDDR4_CHB_CA_0: now reaches U1.L18 (DDR_A14)
- net LPDDR4_CHB_CA_0: now also U18.R2 (CA0_B)
- net LPDDR4_CHA_CKE: now reaches U1.M16 (DDR_A0)
- net LPDDR4_CHA_CKE: now also U18.J4 (CKE0_A)
- net LPDDR4_CHA_CA_1: now reaches U1.M17 (DDR_A3)
- net LPDDR4_CHA_CA_1: now also U18.J2 (CA1_A)
- net LPDDR4_CHA_CLK_N: now reaches U1.M19 (DDR_A5)
- net LPDDR4_CHA_CLK_N: now also U18.J9 (CLK_A_N)
- net LPDDR4_CHA_CA_0: now reaches U1.N16 (DDR_A2)
- net LPDDR4_CHA_CA_0: now also U18.H2 (CA0_A)
- net LPDDR4_CHA_CA_5: now reaches U1.N17 (DDR_A11)
- net LPDDR4_CHA_CA_5: now also U18.J11 (CA5_A)
- net LPDDR4_CHA_CA_4: now reaches U1.N18 (DDR_A10)
- net LPDDR4_CHA_CA_4: now also U18.H11 (CA4_A)
- net LPDDR4_CHA_CLK_P: now reaches U1.N19 (DDR_A4)
- net LPDDR4_CHA_CLK_P: now also U18.J8 (CLK_A_P)
- net LPDDR4_CHA_CA_3: now reaches U1.P18 (DDR_A9)
- net LPDDR4_CHA_CA_3: now also U18.H10 (CA3_A)
- net LPDDR4_CHA_CA_2: now reaches U1.P19 (DDR_A8)
- net LPDDR4_CHA_CA_2: now also U18.H9 (CA2_A)
- net LPDDR4_CHA_CS_N: now reaches U1.T18 (DDR_A6)
- net LPDDR4_CHA_CS_N: now also U18.H4 (CS0_A)
- new net: R83.2, U18.A5 (ZQ0)
- new net: R84.2, U18.A8 (ZQ1)
- no-connect marks 0 -> 20
Other:
- note added: "Bit swap allowed in DQ[15:8]"
- note added: "Bit swap allowed in DQ[7:0]"
- note added: "LPDDR4 channel A"
- note added: "LPDDR4 channel B"
- note added: "LPDDR4 power"
- note added: "Ranks 2/3 NC This is a single rank package"
- note added: "SoC configured for dual channel 16 bit LPDDR4 See 8.7 of AN5489"
- note added: "VDD1 decoupling"
- note added: "VDD2 decoupling"
- note added: "VDDQ decoupling"
