File: pcb/ayrton-mainboard/soc-unused.kicad_sch (KiCad schematic)
At the start: 41 parts, among them U1 STM32MP257FAI3

Commit message: Continued initial system design
Parts:
- removed C1, C13, C14, C15, C16, C17, C18, C19, C2, C20, C21, C22, C23, C24, C25, C26, C27, C28, C29, C3, C30, C31, C32, C33, C34, C35, C36, C37, C38, C39, C4, C40, C5, C6: 1 uF, symbol device:C
- removed C10, C11, C12, C7, C8, C9: 0.47 uF, symbol device:C
- removed U1: STM32MP257FAI3, symbol st-azonenberg:STM32MP257FAI3
- added U1: STM32MP257FAI3, symbol st-azonenberg:STM32MP257FAI3
Other:
- note removed: "Don't bother with analog rail filtering for peripherals we're not using"
- note removed: "TODO: VDDA* VDDIO* VBAT VDD33UCPD VDDA18ON VDD33USB"
- note removed: "VDD (datasheet only calls for 5, do one per pin to be conservative). -44% delta for GRM155R70J105KA12 gives ~660 nF effective"
- note removed: "VDDCORE Datasheet calls for 6 caps Do 7 (one per ball) to be conservative"
- note removed: "VDDCPU"
- note removed: "VDDCSI/DSI/LVDS etc Datasheet calls for 0.1 uF, do 0.47 for commonality w/ other stuff"
- note removed: "VDDGPU Not planning to use the GPU but hook power up just in case we want to play with it"
- note removed: "VDDQDDR 8 caps for 7 power balls, will be fun to lay out"
